File: KiCad/Solar Powered Weather Station.kicad_pcb (KiCad board)
At the start: 2 copper layers, 128.3 x 148.6 mm, 61 parts, among them J1 Solar Charge Controller, J10 Conn_02x06_Odd_Even, J11 External_12V, J12 External_9V, J13 External_5V, J14 External_3V3, J15 WiFi_RX_Switch, J16 WiFi_TX_Switch, J17 Batt_Conn, J2 Solar Panel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

Commit message: Updated PCB
Parts:
- removed J17: Batt_Conn, Connector_PinHeader_2.54mm:PinHeader_1x02_P2.54mm_Vertical
Connections:
- J3 pad 1: Net-(J17-Pad2) -> Net-(J1-Pad3)
Routing:
- net Net-(J17-Pad2): track 8.53 -> 0.00 mm
- net Net-(J1-Pad3): track 52.6 -> 45.9 mm
Other:
- board text removed: "Battery Jumper"
